File: PCB_FILES/MOBILE.kicad_sch (KiCad schematic)
At the start: 33 parts, among them J1 Conn_01x05_Pin, Q1 MMBT3904_C181119, U1 HT7833, U2 ESP32-WROOM-32E-N8R2

Commit message: 3rd commit
Parts:
- removed C1, C12: 10uF, Capacitor_SMD:C_0805_2012Metric, symbol Device:C_Polarized
- removed C10, C3: 33pF, Capacitor_SMD:C_0805_2012Metric, symbol Device:C
- removed C11, C5: 100nF, Capacitor_SMD:C_0805_2012Metric, symbol Device:C
- removed U1: HT7833, easyeda2kicad:SOT-89_L4.5-W2.5-P1.50-LS4.2-BR, symbol easyeda2kicad:HT7833
- added AE1: Antenna, RF_Antenna:Texas_SWRA416_868MHz_915MHz, symbol Device:Antenna
- added C1, C11, C21, C31, C35, C43: 33pF, Capacitor_SMD:C_0805_2012Metric, symbol Device:C_Small
- added C10, C28, C33, C34, C37, C39, C41: 22uF, Capacitor_SMD:C_0805_2012Metric, symbol Device:C_Small
- added C12, C20, C3, C36, C38, C42: 100nF, Capacitor_SMD:C_0805_2012Metric, symbol Device:C_Small
- added C22, C23, C25: 33pF, Capacitor_SMD:C_0805_2012Metric, symbol Device:C
- added C24, C26, C29: TAN 100uF, Capacitor_Tantalum_SMD:CP_EIA-3216-18_Kemet-A, symbol Device:C_Polarized
- added C27, C30, C32, C44: 470uF, Capacitor_SMD:CP_Elec_6.3x7.7, symbol Device:C_Polarized_Small
- added C40: 1uF, Capacitor_SMD:C_0805_2012Metric, symbol Device:C
- added C45, C5: TAN 10uF, Capacitor_Tantalum_SMD:CP_EIA-3216-18_Kemet-A, symbol Device:C_Polarized
- added Card1: SMC-202-6, easyeda2kicad:SIM-SMD_SMC-202-6, symbol easyeda2kicad:SMC-202-6
- added D1: SS34, easyeda2kicad:DO-214AC_L4.3-W2.7-LS5.0-RD, symbol easyeda2kicad:SS34_C84635
- added D2: B540C-13-F, easyeda2kicad:SMC_L7.1-W6.2-LS8.1-RD, symbol easyeda2kicad:B540C-13-F
- added L1, L2: MWSA0603S-4R7MT, easyeda2kicad:IND-SMD_L7.0-W6.6, symbol easyeda2kicad:MCS0630-4R7MPY1
- added L3, L4: CKCS6045-6.8UH/M, easyeda2kicad:IND-SMD_L6.0-W6.0, symbol easyeda2kicad:CKCS6045-6.8UH_M
- added LED1: XL-1606UGC, easyeda2kicad:LED-SMD_L1.7-W1.1-R-RD_GREEN, symbol easyeda2kicad:XL-1606UGC
- added LED2: TZ-P2-0602RTS2-1.2T, easyeda2kicad:LED-SMD_L1.6-W1.2-RD, symbol easyeda2kicad:TZ-P2-0602RTS2-1.2T
- added Q2: SI2333, easyeda2kicad:SOT-23_L2.9-W1.3-P1.90-LS2.4-BR, symbol easyeda2kicad:SI2333_C4748717
- added Q3: AP3404, easyeda2kicad:SOT-23-3_L2.9-W1.3-P1.90-LS2.4-BR-2, symbol easyeda2kicad:AP3404
- added R10, R11, R9: 22R, Resistor_SMD:R_0603_1608Metric, symbol Device:R
- added R12, R22, R23, R26: 1K, Resistor_SMD:R_0603_1608Metric, symbol Device:R
- added R13: 68K, Resistor_SMD:R_0603_1608Metric, symbol Device:R
- added R14: 27K, Resistor_SMD:R_0603_1608Metric, symbol Device:R
- added R16, R27: 100K, Resistor_SMD:R_0603_1608Metric, symbol Device:R
- added R17, R18, R21, R24, R25: 10K, Resistor_SMD:R_0603_1608Metric, symbol Device:R
- added R19: 51K, Resistor_SMD:R_0603_1608Metric, symbol Device:R
- added R20: 1K1, Resistor_SMD:R_0603_1608Metric, symbol Device:R
- added U1: AMS1117-3.3, Package_TO_SOT_SMD:SOT-223-3_TabPin2, symbol Regulator_Linear:AMS1117-3.3
- added U3: M65, easyeda2kicad:XCVR_M65, symbol M65:M65
- added U4: ME2199ASG, easyeda2kicad:SOP-8_L4.9-W3.9-P1.27-LS6.0-BL, symbol easyeda2kicad:ME2199ASG
- added U5: BQ24073RGTR, easyeda2kicad:QFN-16_L3.0-W3.0-P0.50-TL-EP1.7, symbol easyeda2kicad:BQ24073RGTR
Connections:
- net +3V3: now also C11.2, C12.2, C45.1, L4.2
- net +5V: now also U5.13 (IN)
- net EN: now also J1.4 (Pin_4); no longer J1.3 (Pin_3)
- net GND: now also C1.1, C10.1, C11.1, C12.1, C20.1, C21.1, C22.2, C23.2, C24.2, C25.2, C26.2, C27.2, C28.1, C29.2, C3.1, C30.2, C31.1, C32.2, C33.1, C34.2, C35.2, C36.1, C37.1, C38.1, C39.1, C40.1, C41.1, C42.1, C43.1, C44.2, C45.2, C5.2, Card1.10 (GND), Card1.7 (GND), Card1.8 (GND), Card1.9 (GND), LED1.2 (K), Q3.1 (S), R14.2, R16.2, R18.2, R19.2, R20.1, R23.1, R24.1, R25.2, U1.1 (GND), U3.27 (GND), U3.34 (GND), U3.36 (GND), U3.37 (GND), U3.40 (GND), U3.41 (GND), U3.7 (PWRKEY), U4.1 (VSENSE), U4.5 (GND), U5.17 (EP), U5.8 (VSS)
- net IO0: now also J1.1 (Pin_1); no longer J1.4 (Pin_4)
- net UART2_RX: now also U3.17 (TXD)
- net UART2_TX: now also U3.18 (RXD)
- net UOTXD: now also J1.3 (Pin_3); no longer J1.1 (Pin_1)
- net IO17: now reaches U2.28 (IO17)
- net IO17: now also R26.2, R27.2
- new net: R11.2, U3.12 (SIM_RST)
- new net: C29.1, C30.1, C31.2, C38.2, C39.2, D1.2 (A), D2.1 (K), R13.1
- new net: R13.2, R14.1, U4.2 (FB)
- new net: C40.2, U4.3 (VDD)
- new net: Q3.2 (G), U4.7 (EXT)
- new net: D2.2 (A), L2.1, Q3.3 (D)
- new net: R19.1, U5.14 (TMR)
- new net: R16.1, U5.6 (EN1)
- new net: R10.2, U3.13 (SIM_CLK)
- new net: R21.1, U5.7 (~{PGOOD})
- new net: R24.2, U5.1 (TS)
- new net: C10.2, L4.1, U1.2 (VO)
- new net: R9.2, U3.11 (SIM_DATA)
- new net: U3.15 (RESERVED), U3.26 (RESERVED)
- new net: R20.2, U5.12 (ILIM)
- new net: LED2.2 (A), R22.1
- new net: C32.1, C34.1, L3.2, U5.10 (OUT), U5.11 (OUT)
- new net: R23.2, U5.16 (ISET)
- new net: LED1.1 (A), R12.2
- new net: R25.1, U5.15 (TD)
- new net: R18.1, U5.4 (~{CE})
- new net: R17.1, U5.5 (EN2)
- new net: Q2.1 (G), R26.1
- new net 4.2V: D1.1 (C), Q2.2 (S), R27.1
- new net ADC0: U3.9 (ADC0)
- new net BATT+: C33.2, U5.2 (BAT), U5.3 (BAT)
- new net CHR: LED2.1 (K), U5.9 (~{CHG})
- new net DBG_RXD: U3.38 (DBG_RXD)
- new net DBG_TXD: U3.39 (DBG_TXD)
- new net DCD: R12.1, U3.21 (DCD)
- new net GNDA: U3.1 (AGND)
- new net M65_PVR: C20.2, C21.2, C24.1, L1.1, U3.42 (VBAT), U3.43 (VBAT)
- new net MIC+: U3.3 (MICP)
- new net MIC-: U3.4 (MICN)
- new net PCM_CLK: U3.30 (PCM_CLK)
- new net PCM_IN: U3.32 (PCM_IN)
- new net PCM_OUT/MOSI: U3.33 (PCM_OUT)
- new net PCM_SYNC/LCD_CS: U3.31 (PCM_SYNC)
- new net RF_ANT: AE1.1 (A), U3.35 (RF_ANT)
- new net RXD_AUX: U3.28 (RXD_AUX)
- new net SIM_CLK: C23.1, Card1.C3 (CLK), R10.1
- new net SIM_DATA: C22.1, Card1.C7 (I/O), R9.1
- new net SIM_GND: Card1.C5 (GND), U3.10 (SIM_GND)
- new net SIM_RST: C25.1, Card1.C2 (RST), R11.1
- new net SIM_VDD: Card1.C1 (VCC), U3.14 (SIM_VDD)
- new net SPK1+: U3.5 (SPK1P)
- new net SPK1-: U3.6 (SPK1N)
- new net SPK2+: U3.2 (SPK2P)
- new net TXD_AUX: U3.29 (TXD_AUX)
- new net VBAT: C26.1, C27.1, C28.2, L1.2, Q2.3 (D)
- new net VCC: C1.2, C3.2, C35.1, C36.2, C37.2, C41.2, C42.2, C43.2, C44.1, C5.1, L2.2, L3.1, R17.2, R21.2, R22.2, U1.3 (VI), U4.6 (VIN), U4.8 (CE)
- new net VDDA: U3.8 (AVDD)
- new net VDD_EXT: U3.24 (VDD_EXT)
- no-connect marks 14 -> 26
Other:
- note added: "BOOST SECTION"
- note added: "BQ POWER SECTION"
- note added: "BQ'S OUPTUT VOLTAGE TO 3.3V SECTION"
- note added: "M65 MODULE SECTION"
- note added: "POWER CONTROLLED BY ESP32 FOR M65, NFC, GPS SECTION"
- note added: "SIM_CARD"
- note removed: "Voltage Regulator"
